File: Hardware/SparkFun_RTK_Postcard_Portability_Shield.kicad_pcb (KiCad board)
At the start: 2 copper layers, 43.2 x 43.2 mm, 92 parts, among them J1 microSD_Friction, J2 1x10, J3 JST_2mm_LiPo, J4 1x09, SW2 Nav Switch, U1 AP2112K-3.3, U2 MAX17048, U3 MCP73831, U4 PCA9557PW, U5 OLED_1.3"

Commit message: Route board
Parts:
- moved G1 19.3 mm to (213.7, 163.8)
Routing:
- net SD_CD: track 14.6 -> 63.8 mm, vias 2 -> 3
- net 5V: track 25.0 -> 70.9 mm, vias 0 -> 1
- net SCL: track 44.7 -> 74.1 mm, vias 3 -> 5
- net SHLD_POCI: track 15.3 -> 42.8 mm, vias 1 -> 2
- net SHLD_SCK: track 15.5 -> 42.7 mm, vias 2 -> 1
- net SHLD_PICO: track 12.7 -> 36.1 mm, vias 2 -> 1
- net 3V3_EN: track 6.09 -> 29.0 mm, vias 0 -> 2
- net 3.3V_P: track 97.3 -> 118.4 mm
- net SHLD_~{CS}: track 12.5 -> 32.7 mm
- net Net-(D1-K): track 0.00 -> 18.9 mm, vias 0 -> 2
- net SDA: track 47.2 -> 65.9 mm, vias 2 -> 4
- net ~{RESET}_P: track 25.5 -> 39.5 mm
- net GND: track 0.00 -> 10.4 mm, vias 0 -> 49
- net VBATT: track 17.0 -> 23.6 mm
- net Net-(JP1-A): track 0.00 -> 4.14 mm, vias 0 -> 1
- added copper zone on B.Cu, net GND
- added copper zone on F.Cu, net GND
- removed copper zone on B.Cu, net 3.3V_P
- removed copper zone on F.Cu, net 3.3V_P
Other:
- board text added: "Finish: HASL"
- board text removed: "Controlled Impedance: JLC7628"
- board text removed: "Finish: ENIG"
- board text removed: "Inner Copper Weight: 0.5oz"
- board text removed: "No Clean Process"
